File: hardware/sidfi/sidfi.kicad_pcb (KiCad board)
At the start: 2 copper layers, 150 x 65 mm, 45 parts, among them J1 ICSP, J2 SD_CARD, J3 USB_POWER, J4 AUDIO_OUT, J5 LCD_KEYS, Q1 2N3904, U1 74HCT164, U2 74HCT164, U3 MCP1700-3302E_TO92, U4 74HC148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

Commit message: Logo. Redo PCB.
Parts:
- added G***: LOGO, sidfi:logo, F.Cu at (150.2, 79.2)
- added J6: 5V, Connector_PinHeader_2.54mm:PinHeader_1x02_P2.54mm_Vertical, F.Cu at (117.8, 128.8)
- U3: value MCP1700-3302E_TO92 -> MCP1700-3302E
- U5: value PIC32MX270F256B-I_SP -> PIC32MX270F256B
- moved X1 41.4 mm to (201.5, 115.5), turned to 90 degrees
- moved U2 38.3 mm to (167.8, 82.5), turned to 90 degrees
- moved U1 29.2 mm to (167.8, 133.0), turned to 90 degrees
- moved R2 16.2 mm to (193.8, 131.2)
- moved R4 16.1 mm to (188.5, 91.8), turned to 0 degrees
- moved U6 9.26 mm to (183.0, 120.5)
- moved R5 8.94 mm to (200.0, 91.8), turned to 0 degrees
- moved PS1 3.91 mm to (193.8, 82.5), turned to 90 degrees
- moved U5 3.00 mm to (125.2, 120.5)
- moved R1 2.50 mm to (201.5, 131.2)
- moved C2 0.25 mm to (108.8, 107.8)
- moved C3 0.25 mm to (108.8, 128.8)
- moved Y1 0.25 mm to (110.0, 118.2)
Connections:
- J2 pad 2: GND -> Net-(J2-Pad2)
- J2 pad 3: GND -> Net-(J2-Pad3)
Routing:
- net +5V: track 227.5 -> 268.3 mm, vias 5 -> 4
- net 6581_LCD_SDO: track 163.3 -> 124.0 mm, vias 3 -> 2
- net GND: track 44.4 -> 8.67 mm, vias 1 -> 0
- net Net-(U6-Pad6): track 45.2 -> 18.6 mm
- net Net-(C9-Pad1): track 39.4 -> 15.5 mm, vias 1 -> 0
- net +12V: track 98.7 -> 83.2 mm
- net D7: track 60.0 -> 45.0 mm, vias 2 -> 0
- net 6581_LCD_SCK: track 142.1 -> 156.3 mm
- net ICSP_MCLR: track 69.7 -> 55.5 mm
- net A4: track 6.43 -> 19.6 mm, vias 0 -> 1
- net A0: track 16.2 -> 28.1 mm, vias 0 -> 1
- net KEY_1: track 71.1 -> 59.5 mm
- net KEY_2: track 72.5 -> 62.3 mm, vias 2 -> 3
- net KEY_CODE2: track 51.9 -> 42.5 mm, vias 2 -> 1
- net D0: track 59.3 -> 50.2 mm
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Other:
- board text removed: "SIDfi"

Commit message: PCB fixes
Parts:
- moved G*** 2.25 mm to (150.2, 77.0)
Routing:
- net 6581_CS: track 61.2 -> 100.8 mm, vias 1 -> 3
- net SD_CARD_CD: track 60.6 -> 58.6 mm, vias 1 -> 2
- net SD_CARD_CS: track 50.2 -> 48.7 mm, vias 1 -> 2
- net SD_CARD_SDI: track 58.5 -> 57.4 mm, vias 1 -> 2
- net SD_CARD_SDO: track 57.9 -> 57.1 mm, vias 1 -> 2
Other:
- outline, holes or cut-outs redrawn
- board text added: "SIDfi Version 0.1 (c) 2021 Peter Hizalev https://github.com/sidfi/sidfi"
- board text removed: "SIDfi Version 0.1 (c) 2021 Peter Hizalev"

Commit message: Label pins on J1 and J6
Other:
- board text added: "+5V"
- board text added: "MCLR"
- board text added: "PCC"
- board text added: "PGD"
- board text added: "VCC"
